File: device_schematic/negative_supply.kicad_sch (KiCad schematic)
At the start: 4 parts, among them U1 ICL7660S

Commit message: Device schematic update
Parts:
- C1: value Charging capacitor -> 10 µF
- C2: value Negative voltage filtering capacitance -> 10 µF
- JP1: value Negative supply input jumper -> (none)
Changed lines of the file:
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@@
   )
   (symbol (lib_id "Device:C_Polarized") (at 147.32 101.6 0) (unit 1)
-    (in_bom yes) (on_board yes) (fields_autoplaced)
+    (in_bom yes) (on_board yes)
     (property "Reference" "C1" (id 0) (at 151.13 99.4409 0)
       (effects (font (size 1.27 1.27)) (justify left))
     )
-    (property "Value" "Charging capacitor" (id 1) (at 151.13 101.9809 0)
+    (property "Value" "10 µF" (id 1) (at 151.13 101.9809 0)
       (effects (font (size 1.27 1.27)) (justify left))
     )
-    (property "Footprint" "" (id 2) (at 148.2852 105.41 0)
-      (effects (font (size 1.27 1.27)) hide)
+    (property "Footprint" "" (id 2) (at 158.75 105.41 0)
+      (effects (font (size 0 0)) hide)
     )
     (property "Datasheet" "~" (id 3) (at 147.32 101.6 0)
@@
       (effects (font (size 1.27 1.27)) (justify right))
     )
-    (property "Value" "Negative voltage filtering capacitance" (id 1) (at 181.61 103.7589 0)
-      (effects (font (size 1.27 1.27)) (justify right))
+    (property "Value" "10 µF" (id 1) (at 181.61 103.7589 0)
+      (effects (font (size 0 0)) (justify right))
     )
     (property "Footprint" "" (id 2) (at 176.8348 97.79 0)
-      (effects (font (size 1.27 1.27)) hide)
+      (effects (font (size 0 0)) hide)
     )
     (property "Datasheet" "~" (id 3) (at 177.8 101.6 0)
@@
   )
   (symbol (lib_id "Jumper:Jumper_2_Bridged") (at 106.68 91.44 0) (unit 1)
-    (in_bom yes) (on_board yes) (fields_autoplaced)
-    (property "Reference" "JP1" (id 0) (at 106.68 85.09 0))
-    (property "Value" "Negative supply input jumper" (id 1) (at 106.68 87.63 0))
+    (in_bom yes) (on_board yes)
+    (property "Reference" "JP1" (id 0) (at 106.68 88.9 0))
+    (property "Value" "" (id 1) (at 106.68 87.63 0)
+      (effects (font (size 0 0)) hide)
+    )
     (property "Footprint" "" (id 2) (at 106.68 91.44 0)
       (effects (font (size 1.27 1.27)) hide)
