File: device_schematic/signal_processing.kicad_sch (KiCad schematic)
At the start: 0 parts

Commit message: Device schematic update
Parts:
- added C?: 100 nF, symbol Device:C
- added D?: LED, symbol Device:LED
- added D?: 3V3, symbol Device:D_Zener
- added J?: Conn_Coaxial, symbol Connector:Conn_Coaxial
- added JP? (x7): Jumper_2_Bridged, symbol Jumper:Jumper_2_Bridged
- added JP?: Jumper_2_Open, symbol Jumper:Jumper_2_Open
- added R? (x2): 200k, symbol Device:R
- added R?: 330, symbol Device:R
- added R? (x6): 100k, symbol Device:R
- added R?: 100, symbol Device:R
- added SW? (x2): SW_DPST_x2, symbol Switch:SW_DPST_x2
- added U? (x6): MCP6002-xP, symbol Amplifier_Operational:MCP6002-xP
Connections:
- new net: J?.1 (In), JP?.1 (A), R?.1
- new net: C?.1, R?.2, SW?.1 (A)
- new net: C?.2, SW?.2 (B), U?.3 (+)
- new net: R?.1, R?.2, U?.2 (-) (x2)
- new net: JP?.2 (B), R?.2
- new net: D?.1 (K), R?.2 (x2)
- new net: R?.1, R?.2, U?.1 (x2)
- new net: R?.1, R?.1, R?.2, U?.2 (-)
- new net: JP?.1 (A), R?.2, U?.1
- new net: JP?.2 (B), R?.1
- new net: R?.1, U?.1, U?.2 (-)
- new net -5V: JP?.2 (B), JP?.2 (B)
- new net GND: J?.2 (Ext), JP?.1 (A), JP?.2 (B), SW?.1 (A), U?.3 (+), U?.3 (+), U?.3 (+)
- new net NUCLEO 3V3: D?.2 (A), JP?.1 (A)
- new net NUCLEO 5V: JP?.2 (B), JP?.2 (B)
- new net NUCLEO ADC: D?.2 (A), JP?.2 (B)
- new net NUCLEO CHANNEL ENABLED: R?.1, SW?.2 (B)
Other:
- note added: "AC coupling (teoretycznie)"
- note added: "Dzielnik odwracający (3v3 -> -1v65)"
- note added: "Filtr -0.7V do 3.3 V"
- note added: "Odwracający razy pół"
- note added: "Sumator (odwracający)?"
- note added: "bufor odwracający"
